Commit message: Avances en la ejecución

File: description/ros2_control/curtis_motor.ros2_control.xacro (robot description, xacro)
@@ -4,9 +4,10 @@
     <ros2_control name="curtis_motor" type="actuator">
         <hardware>
-            <plugin>caddy_ai2_ros2_control_hardware_curtis_motor_driver/CurtisMotorDriver</plugin>
+            <plugin>caddy_ai2_ros2_control_hardware_curtis_motor_driver/CurtisMotorHardwareInterface</plugin>
+            <param name="can_interface" value="can_motor_drv"/>
             <param name="update_rate" value="${update_rate}"/>
         </hardware>
-        <joint name="curtis_motor">
-            <command_interface name="throttle"/>
+        <joint name="curtis_motor_joint">
+            <command_interface name="velocity"/>
             <state_interface name="velocity"/>
             <state_interface name="current_rms"/>

File: description/urdf/curtis_motor.urdf.xacro (robot description, xacro)
@@ -5,5 +5,38 @@
   <xacro:include filename="$(find caddy_ai2_ros2_control_hardware_curtis_motor_driver)/ros2_control/curtis_motor.ros2_control.xacro" />
   <!-- Used for fixing robot -->
+<!-- Used for fixing robot -->
   <link name="world"/>
+  <joint name="world_to_base" type="fixed">
+    <parent link="world"/>
+    <child link="base_link"/>
+    <origin xyz="0 0 0" rpy="0 0 0"/>
+  </joint>
+  <link name="base_link">
+    <visual>
+      <geometry>
+        <box size="0.1 0.1 0.1"/>
+      </geometry>
+      <material name="blue">
+        <color rgba="0 0 1 1"/>
+      </material>
+    </visual>
+  </link>
+  <joint name="curtis_motor_joint" type="revolute">
+    <parent link="base_link"/>
+    <child link="curtis_motor_link"/>
+    <origin xyz="0 0 0.1" rpy="0 0 0"/>
+    <axis xyz="0 1 0"/>
+    <limit effort="1000" velocity="1000" lower="-3.14" upper="3.14"/>
+  </joint>
+  <link name="curtis_motor_link">
+    <visual>
+      <geometry>
+        <cylinder length="0.1" radius="0.05"/>
+      </geometry>
+      <material name="green">
+        <color rgba="0 1 0 1"/>
+      </material>
+    </visual>
+  </link>
   <xacro:curtis_motor_ros2_control update_rate="$(arg update_rate)"/>
 </robot>
